File: eagle/schaltplan.brd (EAGLE design)
At the start: 160 x 100 mm, 24 parts, among them K1 G5LA1E5DC, K2 G5LA1E5DC, K3 G5LA1E5DC, K4 G5LA1E5DC, K5 G5LA1E5DC, Q1 BC547B, Q2 BC547B, Q3 BC547B, Q4 BC547B, Q5 BC547B, X1 MSTBA8, X2 MSTBA8, X3 MSTBA8

Commit message: fertig #1
Parts:
- moved Q5 67.5 mm to (87.6, 55.9)
- moved D5 67.4 mm to (81.3, 49.5)
- moved K5 67.3 mm to (81.3, 33.0)
- moved X2 64.8 mm to (68.6, 6.35)
- moved Q4 63.7 mm to (69.8, 55.9)
- moved D4 63.6 mm to (63.5, 49.5)
- moved K4 63.5 mm to (63.5, 33.0)
- moved R5 63.5 mm to (86.4, 71.1), turned to 270 degrees
- moved Q3 59.9 mm to (52.1, 55.9)
- moved D3 59.7 mm to (45.7, 49.5)
- moved K3 59.7 mm to (45.7, 33.0)
- moved X1 59.7 mm to (22.9, 6.35)
- moved R4 57.2 mm to (81.3, 71.1), turned to 270 degrees
- moved Q2 56.1 mm to (34.3, 55.9)
- moved D2 55.9 mm to (27.9, 49.5)
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Connections:
- net 0V: now also JP1.25; no longer JP1.20
- net N$27: now also JP1.3; no longer JP1.8
- net N$28: now also JP1.5; no longer JP1.4
- net N$29: now also JP1.9; no longer JP1.1
- net N$30: now also JP1.11; no longer JP1.3
- net N$31: now also JP1.4; no longer JP1.5
- net N$32: now also JP1.8; no longer JP1.9
- net N$33: now also JP1.10; no longer JP1.11
- net N$6: now also JP1.1; no longer JP1.10
- net RASPI_GPIO_22: now also R2.1; no longer R1.1
- net RASPI_GPIO_23: now also R5.1; no longer R2.1
- net RASPI_GPIO_24: now also R4.1; no longer R3.1
- net RASPI_GPIO_25: now also R3.1; no longer R4.1
- net RASPI_GPIO_27: now also R1.1; no longer R5.1
Routing:
- net +5V: track 327.7 -> 213.1 mm, vias 0 -> 2
- net N$27: track 91.8 -> 22.9 mm
- net RASPI_GPIO_23: track 41.2 -> 85.3 mm
- net N$6: track 53.6 -> 10.2 mm
- net N$26: track 5.71 -> 49.2 mm
- net N$5: track 49.7 -> 16.1 mm
- net N$3: track 47.1 -> 16.1 mm
- net N$2: track 47.1 -> 16.1 mm
- net 0V: track 188.9 -> 159.5 mm, vias 0 -> 8
- net N$12: track 59.4 -> 31.1 mm
- net N$7: track 6.98 -> 34.7 mm
- net N$1: track 41.4 -> 16.1 mm
- net N$8: track 6.98 -> 26.7 mm
- net RASPI_GPIO_24: track 59.5 -> 78.4 mm
- net RASPI_GPIO_22: track 30.3 -> 13.5 mm
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Other:
- board size 160 x 100 mm -> 111.7 x 100 mm
