File: eagle/schaltplan.sch (EAGLE design)
At the start: 20 parts, among them K1 G5LA1E5DC, K2 G5LA1E5DC, K3 G5LA1E5DC, K4 G5LA1E5DC, K5 G5LA1E5DC, Q1 BC547B, Q2 BC547B, Q3 BC547B, Q4 BC547B, Q5 BC547B

Commit message: eagle files modified :)
Parts:
- added JP1: (no value), pinhead:PINHD-2X20
- added X1, X2, X3: MSTBA8, con-phoenix-508:MSTBA8
- K1, K2, K3, K4, K5: device relay:G5LE -> relay:G5L
Connections:
- new net N$11: K42.P, X2-3.1
- new net N$12: K12.P, X1-2.1
- new net N$13: K12.O, X1-3.1
- new net N$14: K12.S, X1-1.1
- new net N$15: K22.P, X1-5.1
- new net N$16: K22.O, X1-6.1
- new net N$17: K22.S, X1-4.1
- new net N$18: K32.P, X1-8.1
- new net N$19: K32.O, X2-1.1
- new net N$20: K32.S, X1-7.1
- new net N$21: K42.O, X2-4.1
- new net N$22: K42.S, X2-2.1
- new net N$23: K52.P, X2-6.1
- new net N$24: K52.S, X2-5.1
- new net N$25: K52.O, X2-7.1
- new net N$27: JP1.8, X3-2.1
- new net N$28: JP1.4, X3-3.1
- new net N$29: JP1.1, X3-4.1
- new net N$30: JP1.3, X3-5.1
- new net N$31: JP1.5, X3-6.1
- new net N$32: JP1.9, X3-7.1
- new net N$33: JP1.11, X3-8.1
- new net N$6: JP1.10, X3-1.1
- net +5V: now also JP1.2
- net 0V: now also JP1.20
- net RASPI_GPIO_22: now also JP1.15
- net RASPI_GPIO_23: now also JP1.16
- net RASPI_GPIO_24: now also JP1.18
- net RASPI_GPIO_25: now also JP1.22
- net RASPI_GPIO_27: now also JP1.13
Other:
- moved on the sheet: D1, D2, D3, D4, D5, K1, K2, K3, K4, K5, Q1, Q2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

Commit message: fertig #1
Connections:
- net 0V: now also JP1.25; no longer JP1.20
- net N$27: now also JP1.3; no longer JP1.8
- net N$28: now also JP1.5; no longer JP1.4
- net N$29: now also JP1.9; no longer JP1.1
- net N$30: now also JP1.11; no longer JP1.3
- net N$31: now also JP1.4; no longer JP1.5
- net N$32: now also JP1.8; no longer JP1.9
- net N$33: now also JP1.10; no longer JP1.11
- net N$6: now also JP1.1; no longer JP1.10
- net RASPI_GPIO_22: now also R2.1; no longer R1.1
- net RASPI_GPIO_23: now also R5.1; no longer R2.1
- net RASPI_GPIO_24: now also R4.1; no longer R3.1
- net RASPI_GPIO_25: now also R3.1; no longer R4.1
- net RASPI_GPIO_27: now also R1.1; no longer R5.1
Other:
- moved on the sheet: JP1, X3-1, X3-2, X3-3, X3-4, X3-5, X3-6, X3-7, X3-8
