File: eagle/raspi-gsm-relais.brd (EAGLE design)
At the start: 111.7 x 100 mm, 24 parts, among them K1 G5LA1E5DC, K2 G5LA1E5DC, K3 G5LA1E5DC, K4 G5LA1E5DC, K5 G5LA1E5DC, Q1 BC547B, Q2 BC547B, Q3 BC547B, Q4 BC547B, Q5 BC547B, X1 MSTBA8, X2 MSTBA8, X3 MSTBA8

Commit message: asdf
Parts:
- moved X2 2.54 mm to (71.1, 6.35)
- moved X1 2.54 mm to (25.4, 6.35)
- moved R3 1.27 mm to (77.5, 71.1)
- moved R4 1.27 mm to (82.5, 71.1)
- moved R5 1.27 mm to (87.6, 71.1)
Routing:
- net N$33: track 65.6 -> 72.2 mm
- net N$30: track 54.0 -> 60.1 mm
- net N$32: track 54.6 -> 59.5 mm
- net N$29: track 44.6 -> 49.4 mm
- net 0V: track 159.5 -> 156.5 mm
- net N$31: track 41.8 -> 44.2 mm
- net RASPI_GPIO_24: track 78.4 -> 80.8 mm
- net RASPI_GPIO_23: track 85.3 -> 87.7 mm
- net N$9: track 18.6 -> 16.1 mm
- net N$8: track 26.7 -> 28.8 mm
- net N$28: track 33.1 -> 35.1 mm
- net N$25: track 19.4 -> 17.8 mm
- net N$23: track 33.2 -> 31.7 mm
- net N$24: track 18.6 -> 17.2 mm
- net N$20: track 18.6 -> 17.2 mm
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Other:
- board text added: "raspi-relais v0.1 Dominic Miglar Jan 2014"

Commit message: fertig
Parts:
- added U$1, U$2, U$3, U$4, U$5, U$6: (no value), holes:3,0
- moved D1 8.89 mm to (19.1, 49.5)
- moved D3 8.89 mm to (54.6, 49.5)
- moved D4 8.89 mm to (72.4, 49.5)
- moved D5 8.89 mm to (90.2, 49.5)
- moved K1 8.89 mm to (19.1, 33.0)
- moved K3 8.89 mm to (54.6, 33.0)
- moved K4 8.89 mm to (72.4, 33.0)
- moved K5 8.89 mm to (90.2, 33.0)
- moved Q2 8.89 mm to (43.2, 55.9)
- moved Q3 8.89 mm to (61.0, 55.9)
- moved Q4 8.89 mm to (78.7, 55.9)
- moved Q5 8.89 mm to (96.5, 55.9)
- moved R1 8.89 mm to (68.6, 71.1)
- moved R2 8.89 mm to (73.7, 71.1)
- moved R3 8.89 mm to (86.4, 71.1)
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Routing:
- net N$25: track 17.8 -> 18.6 mm
- net N$16: track 17.0 -> 17.6 mm
- net N$21: track 17.0 -> 17.6 mm
Other:
- board size 111.7 x 100 mm -> 129.5 x 100 mm
