File: eagle/raspi-gsm-relais.sch (EAGLE design)
At the start: 24 parts, among them K1 G5LA1E5DC, K2 G5LA1E5DC, K3 G5LA1E5DC, K4 G5LA1E5DC, K5 G5LA1E5DC, Q1 BC547B, Q2 BC547B, Q3 BC547B, Q4 BC547B, Q5 BC547B, X1 MSTBA8, X2 MSTBA8, X3 MSTBA8

Commit message: added DESCRIPTION
Other:
- note added: "X1-1 ... K1 Schließer X1-2 ... K1 Common X1-3 ... K1 Öffner X1-4 ... K2 Schließer X1-5 ... K2 Common X1-6 ... K2 Öffner X1-7 ... K3 Schließer X1-8 ... K3 Common X2-1 ... K3 Öffner X2-2 ... K4 Schließer X2-3 ... K4 Common X2-4 ... K4 Öffner X2-5 ... K5 Schließer X2-6 ... K5 Common X2-7 ... K5 Öffner"
- note added: "X3-1 ... +3.3V X3-2 ... GPIO2 / I2C SDA X3-3 ... GPIO3 / I2C SCL X3-4 ... GND"
- note added: "X3-5 ... GPIO17 / UART RTS X3-6 ... +5V X3-7 ... GPIO14 / UART TXD X3-8 ... GPIO15 / UART RXD"
- moved on the sheet: K1, K2, K3, K4, K5, X1-1, X1-2, X1-3, X1-4, X1-5, X1-6, X1-7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

Commit message: asdf
Other:
- note added: "0.1"
- note added: "1"
- note added: "AUTHOR:"
- note added: "Dominic Miglar"
- note added: "dominic.miglar@w1r3.net"
Changed lines of the file:
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@@
 <setting verticaltext="up"/>
 </settings>
-<grid distance="0.1" unitdist="inch" unit="inch" style="lines" multiple="1" display="no" altdistance="0.01" altunitdist="inch" altunit="inch"/>
+<grid distance="0.1" unitdist="inch" unit="mm" style="lines" multiple="1" display="yes" altdistance="0.01" altunitdist="inch" altunit="inch"/>
 <layers>
 <layer number="1" name="Top" color="4" fill="1" visible="no" active="no"/>
@@
 X3-7 ... GPIO14 / UART TXD
 X3-8 ... GPIO15 / UART RXD</text>
+<text x="185.42" y="55.88" size="2.54" layer="94">AUTHOR:</text>
+<text x="213.36" y="50.8" size="2.54" layer="94">dominic.miglar@w1r3.net</text>
+<text x="213.36" y="55.88" size="2.54" layer="94">Dominic Miglar</text>
+<text x="222.07" y="36.76" size="2.54" layer="94" font="fixed">1</text>
+<text x="272.85" y="32.65" size="2.54" layer="94">0.1</text>
 </plain>
 <instances>
